File: hardware/instrumentation.kicad_pcb (KiCad board)
At the start: 2 copper layers, 7 parts, among them J1 Conn_01x16_Female, J2 Conn_01x04_Male, U1 ATmega328P-PU, Y1 Crystal

Commit message: pcb updated
Parts:
- removed the C1 at (137.4, 119.1)
- removed the C2 at (137.4, 125.0)
- removed the J1 at (121.7, 100.8)
- removed the J2 at (149.4, 145.3)
- removed the RV1 at (131.3, 102.6)
- removed the U1 at (142.2, 102.6)
- removed the Y1 at (130.6, 124.0)
- added C1: C, Capacitor_THT:C_Disc_D3.8mm_W2.6mm_P2.50mm, F.Cu at (250.1, 112.7)
- added C1: C, Capacitor_THT:C_Disc_D3.8mm_W2.6mm_P2.50mm, F.Cu at (161.7, 111.9)
- added C1: C, Capacitor_THT:C_Disc_D3.8mm_W2.6mm_P2.50mm, F.Cu at (72.6, 111.7)
- added C2: C, Capacitor_THT:C_Disc_D3.8mm_W2.6mm_P2.50mm, F.Cu at (250.4, 94.7)
- added C2: C, Capacitor_THT:C_Disc_D3.8mm_W2.6mm_P2.50mm, F.Cu at (162.0, 93.9)
- added C2: C, Capacitor_THT:C_Disc_D3.8mm_W2.6mm_P2.50mm, F.Cu at (72.8, 93.6)
- added J1: Conn_01x16_Female, Connector_JST:JST_XH_B16B-XH-A_1x16_P2.50mm_Vertical, F.Cu at (229.3, 84.2)
- added J1: Conn_01x16_Female, Connector_JST:JST_XH_B16B-XH-A_1x16_P2.50mm_Vertical, F.Cu at (140.9, 83.5)
- added J1: Conn_01x16_Female, Connector_JST:JST_XH_B16B-XH-A_1x16_P2.50mm_Vertical, F.Cu at (51.7, 83.2)
- added J2: Conn_01x04_Male, Connector:FanPinHeader_1x04_P2.54mm_Vertical, F.Cu at (235.9, 131.5)
- added J2: Conn_01x04_Male, Connector:FanPinHeader_1x04_P2.54mm_Vertical, F.Cu at (147.5, 130.7)
- added J2: Conn_01x04_Male, Connector:FanPinHeader_1x04_P2.54mm_Vertical, F.Cu at (58.3, 130.5)
- added J3: Conn_01x06_Male, Connector_JST:JST_XH_B6B-XH-A_1x06_P2.50mm_Vertical, F.Cu at (254.3, 120.2)
- added J3: Conn_01x06_Male, Connector_JST:JST_XH_B6B-XH-A_1x06_P2.50mm_Vertical, F.Cu at (165.9, 119.4)
- added J3: Conn_01x06_Male, Connector_JST:JST_XH_B6B-XH-A_1x06_P2.50mm_Vertical, F.Cu at (76.7, 119.2)
- added RV1: R_POT, Potentiometer_THT:Potentiometer_ACP_CA9-H5_Horizontal, F.Cu at (241.7, 77.6)
- added RV1: R_POT, Potentiometer_THT:Potentiometer_ACP_CA9-H5_Horizontal, F.Cu at (153.3, 76.9)
- added RV1: R_POT, Potentiometer_THT:Potentiometer_ACP_CA9-H5_Horizontal, F.Cu at (64.2, 76.6)
- added U1: ATmega328P-PU, Package_DIP:DIP-28_W7.62mm, F.Cu at (236.4, 90.8)
- added U1: ATmega328P-PU, Package_DIP:DIP-28_W7.62mm, F.Cu at (148.0, 90.1)
- added U1: ATmega328P-PU, Package_DIP:DIP-28_W7.62mm, F.Cu at (58.8, 89.8)
- added Y1: Crystal, Crystal:Crystal_HC18-U_Vertical, F.Cu at (250.4, 102.3)
- added Y1: Crystal, Crystal:Crystal_HC18-U_Vertical, F.Cu at (162.0, 101.5)
- added Y1: Crystal, Crystal:Crystal_HC18-U_Vertical, F.Cu at (72.8, 101.3)
Routing:
- net (no net): track 0.00 -> 1144.7 mm, vias 0 -> 10
- net +5V: track 0.00 -> 101.8 mm
- net Net-(J1-Pad6): track 0.00 -> 86.9 mm
- net Net-(J3-Pad1): track 0.00 -> 49.2 mm
- net Net-(J1-Pad4): track 0.12 -> 46.5 mm
- net Net-(C1-Pad1): track 13.3 -> 57.8 mm
- net Net-(C2-Pad1): track 12.3 -> 45.8 mm
- net Net-(J1-Pad8): track 25.3 -> 0.00 mm
- net Net-(J1-Pad7): track 25.0 -> 0.00 mm
- net Net-(J1-Pad9): track 25.0 -> 0.00 mm
- net Net-(J1-Pad10): track 24.9 -> 0.00 mm
- net Net-(J1-Pad15): track 24.1 -> 0.00 mm
- net Net-(J2-Pad1): track 20.7 -> 44.2 mm
- net GND: track 0.00 -> 18.4 mm, vias 0 -> 5
- net Net-(J1-Pad11): track 24.9 -> 9.56 mm
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- added copper zone on F.Cu, net (none)
- added copper zone on F.Cu, net GND
Other:
- board outline added: 229.9 x 73.2 mm
- board text added: "Deux V.beta"
