File: hardware/instrumentation.sch (KiCad schematic (older format))
At the start: 8 parts, among them J1 Conn_01x16_Female, J2 Conn_01x04_Male, J3 AVR-ISP-6, U1 ATmega328P-PU, Y1 Crystal

Commit message: pcb updated
Parts:
- removed J3: AVR-ISP-6, Connector_IDC:IDC-Header_2x03_P2.54mm_Vertical, symbol instrumentation-rescue:AVR-ISP-6-Connector
- added J3: Conn_01x06_Male, Connector_JST:JST_XH_B6B-XH-A_1x06_P2.50mm_Vertical, symbol Connector:Conn_01x06_Male
- U1: symbol instrumentation-rescue:ATmega328P-PU-MCU_Microchip_ATmega -> MCU_Microchip_ATmega:ATmega328P-PU
Connections:
- net +5V: now also J3.6 (Pin_6)
- net GND: now also J1.10 (Pin_10), J1.7 (Pin_7), J1.8 (Pin_8), J1.9 (Pin_9), J3.5 (Pin_5)
- net at U1.5 (PD3): no longer J1.10 (Pin_10)
- net at U1.2 (PD0): no longer J1.7 (Pin_7)
- net at U1.3 (PD1): no longer J1.8 (Pin_8)
- net at U1.4 (PD2): no longer J1.9 (Pin_9)
- net at U1.1 (~RESET~/PC6): now also J3.1 (Pin_1)
- net at U1.17 (PB3): now also J3.4 (Pin_4)
- net at U1.18 (PB4): now also J3.3 (Pin_3)
- net at U1.19 (PB5): now also J3.2 (Pin_2)
Changed lines of the file:
@@
 EESchema Schematic File Version 4
-LIBS:instrumentation-cache
-EELAYER 26 0
+EELAYER 30 0
 EELAYER END
 $Descr A4 11693 8268
@@
 	6250 2750 5850 2750
 Wire Wire Line
-	3950 3300 2800 3300
-Wire Wire Line
-	2800 3300 2800 5800
-Wire Wire Line
-	2800 5800 6300 5800
-Wire Wire Line
-	6300 5800 6300 4350
-Wire Wire Line
-	6300 4350 5850 4350
-Wire Wire Line
-	5850 4450 6200 4450
-Wire Wire Line
-	6200 4450 6200 5750
-Wire Wire Line
-	6200 5750 2850 5750
-Wire Wire Line
-	2850 5750 2850 3400
-Wire Wire Line
-	2850 3400 3950 3400
-Wire Wire Line
-	5850 4550 6100 4550
-Wire Wire Line
-	6100 4550 6100 5650
-Wire Wire Line
-	6100 5650 2900 5650
-Wire Wire Line
-	2900 5650 2900 3500
-Wire Wire Line
-	2900 3500 3950 3500
-Wire Wire Line
-	3950 3600 2950 3600
-Wire Wire Line
-	2950 3600 2950 5600
-Wire Wire Line
-	2950 5600 6050 5600
-Wire Wire Line
-	6050 5600 6050 4650
-Wire Wire Line
-	6050 4650 5850 4650
-Wire Wire Line
-	5850 4750 6350 4750
-Wire Wire Line
-	6350 4750 6350 5900
-Wire Wire Line
-	6350 5900 3150 5900
-Wire Wire Line
-	3150 5900 3150 3700
-Wire Wire Line
-	3150 3700 3950 3700
-Wire Wire Line
-	3950 3800 2650 3800
-Wire Wire Line
-	2650 3800 2650 6000
-Wire Wire Line
-	2650 6000 6550 6000
-Wire Wire Line
-	6550 6000 6550 4800
-Wire Wire Line
-	6550 4800 5850 4800
-Wire Wire Line
-	5850 4800 5850 4850
-Wire Wire Line
-	5850 4950 6800 4950
-Wire Wire Line
-	6800 4950 6800 5400
-Wire Wire Line
-	6800 5400 3300 5400
-Wire Wire Line
-	3300 5400 3300 3900
-Wire Wire Line
-	3300 3900 3950 3900
-Wire Wire Line
-	3950 4000 3400 4000
-Wire Wire Line
-	3400 4000 3400 5500
-Wire Wire Line
-	3400 5500 5850 5500
-Wire Wire Line
-	5850 5500 5850 5050
-Wire Wire Line
 	6050 3250 6050 3150
 Wire Wire Line
@@
 	5350 6300 5350 6450
 Wire Wire Line
-	5850 3150 5950 3150
-Wire Wire Line
-	5950 3150 5950 2900
-Wire Wire Line
-	5950 2900 8000 2900
-Wire Wire Line
-	8000 2900 8000 3500
-Wire Wire Line
-	8250 3050 8250 3400
-Wire Wire Line
-	5850 3050 8250 3050
-Wire Wire Line
-	5850 4150 8250 4150
-Wire Wire Line
-	8250 4150 8250 3600
-Wire Wire Line
-	5850 2950 8900 2950
-Wire Wire Line
-	8900 2950 8900 3500
-Wire Wire Line
 	5850 3950 7800 3950
 Wire Wire Line
@@
 $EndComp
 $Comp
-L power:+5V #PWR0103
-U 1 1 5E5A47D6
-P 9250 3000
-F 0 "#PWR0103" H 9250 2850 50  0001 C CNN
-F 1 "+5V" H 9265 3173 50  0000 C CNN
-F 2 "" H 9250 3000 50  0001 C CNN
-F 3 "" H 9250 3000 50  0001 C CNN
-	1    9250 3000
-	1    0    0    -1
-$EndComp
-$Comp
 L power:+5V #PWR0104
 U 1 1 5E5A6ABC
@@
 $EndComp
 $Comp
-L instrumentation-rescue:ATmega328P-PU-MCU_Microchip_ATmega U1
+L MCU_Microchip_ATmega:ATmega328P-PU U1
 U 1 1 5E4D81ED
 P 5250 3850
@@
 F 3 "http://ww1.microchip.com/downloads/en/DeviceDoc/ATmega328_P%20AVR%20MCU%20with%20picoPower%20Technology%20Data%20Sheet%2040001984A.pdf" H 5250 3850 50  0001 C CNN
 	1    5250 3850
-	1    0    0    -1
-$EndComp
-$Comp
-L power:GND #PWR0107
-U 1 1 5E5AE1CD
-P 9250 3900
-F 0 "#PWR0107" H 9250 3650 50  0001 C CNN
-F 1 "GND" H 9255 3727 50  0000 C CNN
-F 2 "" H 9250 3900 50  0001 C CNN
-F 3 "" H 9250 3900 50  0001 C CNN
-	1    9250 3900
 	1    0    0    -1
 $EndComp
@@
 	0    -1   -1   0
 $EndComp
-$Comp
-L instrumentation-rescue:AVR-ISP-6-Connector J3
-U 1 1 5E5B7DA1
-P 9350 3500
-F 0 "J3" H 9021 3596 50  0000 R CNN
-F 1 "AVR-ISP-6" H 9021 3505 50  0000 R CNN
-F 2 "Connector_IDC:IDC-Header_2x03_P2.54mm_Vertical" V 9100 3550 50  0001 C CNN
-F 3 " ~" H 8075 2950 50  0001 C CNN
-	1    9350 3500
-	1    0    0    -1
-$EndComp
-Wire Wire Line
-	8900 3500 8750 3500
-Wire Wire Line
-	8500 3500 8500 4250
-Wire Wire Line
-	8500 4250 9900 4250
-Wire Wire Line
-	9900 4250 9900 3500
-Wire Wire Line
-	9900 3500 9750 3500
-Wire Wire Line
-	8000 3500 8500 3500
-Wire Wire Line
-	9750 3300 9750 2850
-Wire Wire Line
-	9750 2850 8400 2850
-Wire Wire Line
-	8400 2850 8400 3400
-Wire Wire Line
-	8400 3400 8250 3400
-Wire Wire Line
-	8750 3500 8750 4200
-Wire Wire Line
-	8750 4200 10150 4200
-Wire Wire Line
-	10150 4200 10150 3400
-Wire Wire Line
-	10150 3400 9750 3400
-Wire Wire Line
-	8250 3600 9750 3600
 Wire Wire Line
 	5250 2200 5250 2350
 $Comp
-L power:+5V #PWR?
+L power:+5V #PWR0113
 U 1 1 5E5D38A1
 P 3950 4100
-F 0 "#PWR?" H 3950 3950 50  0001 C CNN
+F 0 "#PWR0113" H 3950 3950 50  0001 C CNN
 F 1 "+5V" V 3965 4228 50  0000 L CNN
 F 2 "" H 3950 4100 50  0001 C CNN
@@
 $EndComp
 $Comp
-L power:GND #PWR?
+L power:GND #PWR0114
 U 1 1 5E4C1D1F
 P 5450 6450
-F 0 "#PWR?" H 5450 6200 50  0001 C CNN
+F 0 "#PWR0114" H 5450 6200 50  0001 C CNN
 F 1 "GND" H 5455 6277 50  0000 C CNN
 F 2 "" H 5450 6450 50  0001 C CNN
@@
 	-1   0    0    1
 $EndComp
+$Comp
+L power:GND #PWR0115
+U 1 1 5E5E77B5
+P 3950 3300
+F 0 "#PWR0115" H 3950 3050 50  0001 C CNN
+F 1 "GND" V 3955 3172 50  0000 R CNN
+F 2 "" H 3950 3300 50  0001 C CNN
+F 3 "" H 3950 3300 50  0001 C CNN
+	1    3950 3300
+	0    1    1    0
+$EndComp
+$Comp
+L power:GND #PWR0116
+U 1 1 5E5E830A
+P 3950 3400
+F 0 "#PWR0116" H 3950 3150 50  0001 C CNN
+F 1 "GND" V 3955 3272 50  0000 R CNN
+F 2 "" H 3950 3400 50  0001 C CNN
+F 3 "" H 3950 3400 50  0001 C CNN
+	1    3950 3400
+	0    1    1    0
+$EndComp
+$Comp
+L power:GND #PWR0117
+U 1 1 5E5E89F8
+P 3950 3500
+F 0 "#PWR0117" H 3950 3250 50  0001 C CNN
+F 1 "GND" V 3955 3372 50  0000 R CNN
+F 2 "" H 3950 3500 50  0001 C CNN
+F 3 "" H 3950 3500 50  0001 C CNN
+	1    3950 3500
+	0    1    1    0
+$EndComp
+$Comp
+L power:GND #PWR0118
+U 1 1 5E5E8E71
+P 3950 3600
+F 0 "#PWR0118" H 3950 3350 50  0001 C CNN
+F 1 "GND" V 3955 3472 50  0000 R CNN
+F 2 "" H 3950 3600 50  0001 C CNN
+F 3 "" H 3950 3600 50  0001 C CNN
+	1    3950 3600
+	0    1    1    0
+$EndComp
+Wire Wire Line
+	3950 3700 3150 3700
+Wire Wire Line
+	3150 3700 3150 5400
+Wire Wire Line
+	3150 5400 6100 5400
+Wire Wire Line
+	6100 5400 6100 4750
+Wire Wire Line
+	6100 4750 5850 4750
+Wire Wire Line
+	3950 3800 3200 3800
+Wire Wire Line
+	3200 3800 3200 5500
+Wire Wire Line
+	3200 5500 6200 5500
+Wire Wire Line
+	6200 5500 6200 4850
+Wire Wire Line
+	6200 4850 5850 4850
+Wire Wire Line
+	3950 3900 3300 3900
+Wire Wire Line
+	3300 3900 3300 5600
+Wire Wire Line
+	3300 5600 6350 5600
+Wire Wire Line
+	6350 5600 6350 4950
+Wire Wire Line
+	6350 4950 5850 4950
+Wire Wire Line
+	3950 4000 3350 4000
+Wire Wire Line
+	3350 4000 3350 5800
+Wire Wire Line
+	3350 5800 6450 5800
+Wire Wire Line
+	6450 5800 6450 5050
+Wire Wire Line
+	6450 5050 5850 5050
+$Comp
+L Connector:Conn_01x06_Male J3
+U 1 1 5E6553F3
+P 8600 3450
+F 0 "J3" H 8572 3332 50  0000 R CNN
+F 1 "Conn_01x06_Male" H 8572 3423 50  0000 R CNN
+F 2 "Connector_JST:JST_XH_B6B-XH-A_1x06_P2.50mm_Vertical" H 8600 3450 50  0001 C CNN
+F 3 "~" H 8600 3450 50  0001 C CNN
+	1    8600 3450
+	-1   0    0    1
+$EndComp
+$Comp
+L power:+5V #PWR0103
+U 1 1 5E673F21
+P 8400 3150
+F 0 "#PWR0103" H 8400 3000 50  0001 C CNN
+F 1 "+5V" H 8415 3323 50  0000 C CNN
+F 2 "" H 8400 3150 50  0001 C CNN
+F 3 "" H 8400 3150 50  0001 C CNN
+	1    8400 3150
+	1    0    0    -1
+$EndComp
+$Comp
+L power:GND #PWR0107
+U 1 1 5E6744AE
+P 8400 3250
+F 0 "#PWR0107" H 8400 3000 50  0001 C CNN
+F 1 "GND" H 8405 3077 50  0000 C CNN
+F 2 "" H 8400 3250 50  0001 C CNN
+F 3 "" H 8400 3250 50  0001 C CNN
+	1    8400 3250
+	0    1    1    0
+$EndComp
+Wire Wire Line
+	5900 3150 5850 3150
+Wire Wire Line
+	8400 3650 5950 3650
+Wire Wire Line
+	5950 3650 5950 4150
+Wire Wire Line
+	5950 4150 5850 4150
+Wire Wire Line
+	8400 3350 7400 3350
+Wire Wire Line
+	7400 3350 7400 2950
+Wire Wire Line
+	7400 2950 5850 2950
+Wire Wire Line
+	8400 3450 7550 3450
+Wire Wire Line
+	7550 3450 7550 3050
+Wire Wire Line
+	7550 3050 5850 3050
+Wire Wire Line
+	8400 3550 7300 3550
+Wire Wire Line
+	7300 3550 7300 2850
+Wire Wire Line
+	7300 2850 5900 2850
+Wire Wire Line
+	5900 2850 5900 3150
 $EndSCHEMATC
