File: hardware/instrumentation.sch (KiCad schematic (older format))
At the start: 8 parts, among them J1 Conn_01x16_Female, J2 Conn_01x04_Male, J3 Conn_01x06_Male, U1 ATmega328P-PU, Y1 16 Mhz Crystal

Commit message: Project Submission Done/
Parts:
- added R?: R, symbol Device:R
Connections:
- net +5V: now also R?.2
- net GND: now also R?.1
Changed lines of the file:
@@
 Wire Wire Line
 	5900 2850 5900 3150
+$Comp
+L Device:R R?
+U 1 1 5E5CCA80
+P 8550 4100
+F 0 "R?" H 8620 4146 50  0000 L CNN
+F 1 "R" H 8620 4055 50  0000 L CNN
+F 2 "" V 8480 4100 50  0001 C CNN
+F 3 "~" H 8550 4100 50  0001 C CNN
+	1    8550 4100
+	1    0    0    -1
+$EndComp
+$Comp
+L power:GND #PWR?
+U 1 1 5E5CCCA2
+P 8550 3950
+F 0 "#PWR?" H 8550 3700 50  0001 C CNN
+F 1 "GND" H 8555 3777 50  0000 C CNN
+F 2 "" H 8550 3950 50  0001 C CNN
+F 3 "" H 8550 3950 50  0001 C CNN
+	1    8550 3950
+	0    1    1    0
+$EndComp
+$Comp
+L power:+5V #PWR?
+U 1 1 5E5CCE8A
+P 8550 4250
+F 0 "#PWR?" H 8550 4100 50  0001 C CNN
+F 1 "+5V" V 8565 4378 50  0000 L CNN
+F 2 "" H 8550 4250 50  0001 C CNN
+F 3 "" H 8550 4250 50  0001 C CNN
+	1    8550 4250
+	0    -1   -1   0
+$EndComp
 $EndSCHEMATC
